File: hw/frontend/daisho_rs232_fe/rs232_fe/rs232_fe.kicad_pcb (KiCad board)
At the start: 4 copper layers, 100 x 100 mm, 169 parts, among them J1 SAMTEC_QSH-090-D, J2 DB9, J3 DB9, J4 DB9, J5 DB9, P1 CONN_2, P10 CONN_3, P11 CONN_3, P12 CONN_3, P13 CONN_8X2, P14 CONN_3, P2 CONN_3, P3 CONN_3, P4 CONN_3, P5 CONN_3, P6 CONN_8X2, P7 CONN_2, P8 CONN_2, P9 CONN_3, Q1 MUN5212DW1, Q10 MUN5212DW1, Q11 MUN5212DW1, Q12 MUN5212DW1, Q13 MUN5212DW1, Q14 MUN5212DW1, Q15 MUN5212DW1, Q16 MUN5212DW1, Q2 MUN5212DW1, Q3 MUN5212DW1, Q4 MUN5212DW1, Q5 MUN5212DW1, Q6 MUN5212DW1, Q7 MUN5212DW1, Q8 MUN5212DW1, Q9 MUN5212DW1, U1 24C08, U2 TRSF3243, U3 TRS3237E, U4 TRSF3243, U5 TRS3237E, U6 MIC5318, U7 MIC5318

Commit message: rs232: gerber options
Routing:
- net REG_3V3_LED: track 204.7 -> 178.4 mm
- net REG_3V3: track 192.0 -> 191.4 mm
